Commit message: anfang der echten vis

File: Data/spirob.urdf (robot description, URDF)
Before this commit: robot spirob, 21 links, 20 joints
Links:
- removed link seg_13
- removed link seg_14
- removed link seg_15
- removed link seg_16
- removed link seg_17
- removed link seg_18
- removed link seg_19
- added link seg_-1, mass 0.102123036; visual mesh filename=meshes/seg_-1.stl scale=0.001 0.001 0.001
- link seg_0: mass 0.000618575415 -> 0.00310262138; geometry visual mesh filename=meshes/seg_0.stl scale=0.001 0.001 0.001
- link seg_1: mass 0.000809310813 -> 0.00405930298; geometry visual mesh filename=meshes/seg_1.stl scale=0.001 0.001 0.001
- link seg_10: mass 0.00909116481 -> 0.0455990354; geometry visual mesh filename=meshes/seg_10.stl scale=0.001 0.001 0.001
- link seg_11: mass 0.0118943912 -> 0.0596593261; geometry visual mesh filename=meshes/seg_11.stl scale=0.001 0.001 0.001
- link seg_12: mass 0.0155619819 -> 0.0780550545; geometry visual mesh filename=meshes/seg_12.stl scale=0.001 0.001 0.001
- link seg_2: mass 0.00105885875 -> 0.00531097376; geometry visual mesh filename=meshes/seg_2.stl scale=0.001 0.001 0.001
- link seg_3: mass 0.00138535386 -> 0.0069485925; geometry visual mesh filename=meshes/seg_3.stl scale=0.001 0.001 0.001
- link seg_4: mass 0.0018125225 -> 0.00909116481; geometry visual mesh filename=meshes/seg_4.stl scale=0.001 0.001 0.001
- link seg_5: mass 0.00237140698 -> 0.0118943912; geometry visual mesh filename=meshes/seg_5.stl scale=0.001 0.001 0.001
- link seg_6: mass 0.00310262138 -> 0.0155619819; geometry visual mesh filename=meshes/seg_6.stl scale=0.001 0.001 0.001
- link seg_7: mass 0.00405930298 -> 0.0203604604; geometry visual mesh filename=meshes/seg_7.stl scale=0.001 0.001 0.001
- link seg_8: mass 0.00531097376 -> 0.0266385316; geometry visual mesh filename=meshes/seg_8.stl scale=0.001 0.001 0.001
- link seg_9: mass 0.0069485925 -> 0.0348524224; geometry visual mesh filename=meshes/seg_9.stl scale=0.001 0.001 0.001
Joints:
- removed joint j_13
- removed joint j_14
- removed joint j_15
- removed joint j_16
- removed joint j_17
- removed joint j_18
- joint fixed_root: child seg_19 -> seg_-1
- joint j_0: origin xyz=0 0 0.00615045907 rpy=0 0 0 -> xyz=0 0 0.0105281705 rpy=0 0 0
- joint j_1: origin xyz=0 0 0.00672690191 rpy=0 0 0 -> xyz=0 0 0.0115149079 rpy=0 0 0
- joint j_10: origin xyz=0 0 0.0150654864 rpy=0 0 0 -> xyz=0 0 0.0257886455 rpy=0 0 0
- joint j_11: origin xyz=0 0 0.0164774772 rpy=0 0 0 -> xyz=0 0 0.0282056489 rpy=0 0 0
- joint j_12: origin xyz=0 0 0.0180218049 rpy=0 0 0 -> xyz=0 0 0.0308491824 rpy=0 0 0; parent seg_13 -> seg_-1
- joint j_2: origin xyz=0 0 0.00735737102 rpy=0 0 0 -> xyz=0 0 0.012594126 rpy=0 0 0
- joint j_3: origin xyz=0 0 0.00804692994 rpy=0 0 0 -> xyz=0 0 0.0137744921 rpy=0 0 0
- joint j_4: origin xyz=0 0 0.00880111676 rpy=0 0 0 -> xyz=0 0 0.0150654864 rpy=0 0 0
- joint j_5: origin xyz=0 0 0.00962598865 rpy=0 0 0 -> xyz=0 0 0.0164774772 rpy=0 0 0
- joint j_6: origin xyz=0 0 0.0105281705 rpy=0 0 0 -> xyz=0 0 0.0180218049 rpy=0 0 0
- joint j_7: origin xyz=0 0 0.0115149079 rpy=0 0 0 -> xyz=0 0 0.0197108723 rpy=0 0 0
- joint j_8: origin xyz=0 0 0.012594126 rpy=0 0 0 -> xyz=0 0 0.0215582452 rpy=0 0 0
- joint j_9: origin xyz=0 0 0.0137744921 rpy=0 0 0 -> xyz=0 0 0.0235787605 rpy=0 0 0

Commit message: update visual

File: Data/spirob.urdf (robot description, URDF)
Before this commit: robot spirob, 15 links, 14 joints
Joints:
- joint j_0: origin xyz=0 0 0.0105281705 rpy=0 0 0 -> xyz=0 0 0.018249 rpy=0 0 0
- joint j_1: origin xyz=0 0 0.0115149079 rpy=0 0 0 -> xyz=0 0 0.02002 rpy=0 0 0
- joint j_10: origin xyz=0 0 0.0257886455 rpy=0 0 0 -> xyz=0 0 0.046074 rpy=0 0 0
- joint j_11: origin xyz=0 0 0.0282056489 rpy=0 0 0 -> xyz=0 0 0.050545 rpy=0 0 0
- joint j_12: origin xyz=0 0 0.0308491824 rpy=0 0 0 -> xyz=0 0 0.05545 rpy=0 0 0
- joint j_2: origin xyz=0 0 0.012594126 rpy=0 0 0 -> xyz=0 0 0.021963 rpy=0 0 0
- joint j_3: origin xyz=0 0 0.0137744921 rpy=0 0 0 -> xyz=0 0 0.024094 rpy=0 0 0
- joint j_4: origin xyz=0 0 0.0150654864 rpy=0 0 0 -> xyz=0 0 0.026432 rpy=0 0 0
- joint j_5: origin xyz=0 0 0.0164774772 rpy=0 0 0 -> xyz=0 0 0.028997 rpy=0 0 0
- joint j_6: origin xyz=0 0 0.0180218049 rpy=0 0 0 -> xyz=0 0 0.031811 rpy=0 0 0
- joint j_7: origin xyz=0 0 0.0197108723 rpy=0 0 0 -> xyz=0 0 0.034897 rpy=0 0 0
- joint j_8: origin xyz=0 0 0.0215582452 rpy=0 0 0 -> xyz=0 0 0.038284 rpy=0 0 0
- joint j_9: origin xyz=0 0 0.0235787605 rpy=0 0 0 -> xyz=0 0 0.041999 rpy=0 0 0
